Commit message: rectify robot model

File: resources/robots/wheel_legged_fyt/urdf/wheel_legged_v4.urdf (robot description, URDF)
Before this commit: robot wheel_legged_v4, 7 links, 6 joints
Links:
- link base_link: geometry collision mesh filename=package://wheel_legged_v4_ready2use_test/meshes/base_link.S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; visual mesh filename=package://wheel_legged_v4_ready2use_test/meshes/base_link.S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
- link left_leg_link: geometry collision mesh filename=package://wheel_legged_v4_ready2use_test/meshes/left_leg_li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; visual mesh filename=package://wheel_legged_v4_ready2use_test/meshes/left_leg_li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
- link left_thigh_link: geometry collision mesh filename=package://wheel_legged_v4_ready2use_test/meshes/left_thigh_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; visual mesh filename=package://wheel_legged_v4_ready2use_test/meshes/left_thigh_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
- link left_wheel_link: geometry collision mesh filename=package://wheel_legged_v4_ready2use_test/meshes/left_wheel_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; visual mesh filename=package://wheel_legged_v4_ready2use_test/meshes/left_wheel_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
- link right_leg_link: geometry collision mesh filename=package://wheel_legged_v4_ready2use_test/meshes/right_leg_l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; visual mesh filename=package://wheel_legged_v4_ready2use_test/meshes/right_leg_l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
- link right_thigh_link: geometry collision mesh filename=package://wheel_legged_v4_ready2use_test/meshes/right_thigh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; visual mesh filename=package://wheel_legged_v4_ready2use_test/meshes/right_thigh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
- link right_wheel_link: geometry collision mesh filename=package://wheel_legged_v4_ready2use_test/meshes/right_wheel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; visual mesh filename=package://wheel_legged_v4_ready2use_test/meshes/right_wheel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
Joints:
- joint left_leg_joint: limit lower=-1 upper=0.65 effort=30 velocity=1000 -> lower=-0.7 upper=1.2 effort=30 velocity=1000; origin xyz=-0.18482 0.099701 0.018 rpy=0 0 0 -> xyz=-0.21 0.0 0.018 rpy=0 0 0
- joint left_wheel_joint: origin xyz=0.21482 0.12787 0.022043 rpy=0 0 0 -> xyz=0.0 0.25 0.022043 rpy=0 0 0
- joint right_leg_joint: limit lower=-0.5 upper=1.05 effort=30 velocity=1000 -> lower=-1.2 upper=0.7 effort=30 velocity=1000; origin xyz=-0.19554 -0.076574 0.018 rpy=0 0 0 -> xyz=-0.21 0.0 0.018 rpy=0 0 0
- joint right_wheel_joint: origin xyz=0.21678 -0.12453 0.022043 rpy=0 0 0 -> xyz=0.0 -0.25 0.022043 rpy=0 0 0

File: resources/robots/wheel_legged_fyt/urdf/wheel_legged_v4_isaac.urdf (robot description, URDF)
Before this commit: robot wheel_legged_v4, 7 links, 6 joints
Joints:
- joint left_leg_joint: limit lower=-1 upper=0.65 effort=30 velocity=1000 -> lower=-0.7 upper=1.2 effort=30 velocity=1000; origin xyz=-0.18482 0.099701 0.018 rpy=0 0 0 -> xyz=-0.21 0.0 0.018 rpy=0 0 0
- joint left_wheel_joint: origin xyz=0.21482 0.12787 0.022043 rpy=0 0 0 -> xyz=0.0 0.25 0.022043 rpy=0 0 0
- joint right_leg_joint: limit lower=-0.5 upper=1.05 effort=30 velocity=1000 -> lower=-1.2 upper=0.7 effort=30 velocity=1000; origin xyz=-0.19554 -0.076574 0.018 rpy=0 0 0 -> xyz=-0.21 0.0 0.018 rpy=0 0 0
- joint right_wheel_joint: origin xyz=0.21678 -0.12453 0.022043 rpy=0 0 0 -> xyz=0.0 -0.25 0.022043 rpy=0 0 0
