Commit message: fix leg_joint rotation axis bug

File: resources/robots/wheel_legged_fyt/urdf/wheel_legged_v4_isaac.urdf (robot description, URDF)
Before this commit: robot wheel_legged_v4, 7 links, 6 joints
Joints:
- joint left_leg_joint: axis 0 0 -1 -> 0 0 1; limit lower=-0.7 upper=1.2 effort=30 velocity=1000 -> lower=-1.2 upper=0.7 effort=30 velocity=1000
- joint left_wheel_joint: limit effort=5 velocity=1000 -> effort=4.5 velocity=1000
- joint right_leg_joint: axis 0 0 -1 -> 0 0 1; limit lower=-1.2 upper=0.7 effort=30 velocity=1000 -> lower=-0.7 upper=1.2 effort=30 velocity=1000
- joint right_wheel_joint: limit effort=5 velocity=1000 -> effort=4.5 velocity=1000

Commit message: add annotations

File: resources/robots/wheel_legged_fyt/urdf/wheel_legged_v4_isaac.urdf (robot description, URDF)
Before this commit: robot wheel_legged_v4, 7 links, 6 joints
Links:
- link left_leg_link: mass 0.2756 -> 0.32
- link left_thigh_link: mass 0.450 -> 0.3
- link right_leg_link: mass 0.2756 -> 0.32
- link right_thigh_link: mass 0.450 -> 0.3

Commit message: fix: stabilize FYT VMC exploration

File: resources/robots/wheel_legged_fyt/urdf/wheel_legged_v4_isaac.urdf (robot description, URDF)
Before this commit: robot wheel_legged_v4, 7 links, 6 joints
Joints:
- joint left_thigh_joint: type continuous -> revolute
- joint right_thigh_joint: type continuous -> revolute

Commit message: add reading annotations

File: resources/robots/wheel_legged_fyt/urdf/wheel_legged_v4_isaac.urdf (robot description, URDF)
Before this commit: robot wheel_legged_v4, 7 links, 6 joints
Joints:
- joint left_wheel_joint: type continuous -> revolute
- joint right_wheel_joint: type continuous -> revolute
