Commit message: fix: align whole robot joint limits

File: resources/robots/wheel_legged_fyt_whole/urdf/wheel_legged_fyt_whole.urdf (robot description, URDF)
Before this commit: robot wheel_legged_fyt_whole, 7 links, 6 joints
Joints:
- joint left_leg_joint: limit lower=-3.14 upper=3.14 effort=100 velocity=100 -> lower=-1.2 upper=0.7 effort=30 velocity=1000
- joint left_thigh_joint: limit lower=-3.14 upper=3.14 effort=100 velocity=100 -> lower=-3.14 upper=3.14 effort=30 velocity=1000
- joint left_wheel_joint: limit lower=-3.14 upper=3.14 effort=100 velocity=100 -> effort=4.5 velocity=1000
- joint right_leg_joint: limit lower=-3.14 upper=3.14 effort=100 velocity=100 -> lower=-0.7 upper=1.2 effort=30 velocity=1000
- joint right_thigh_joint: limit lower=-3.14 upper=3.14 effort=100 velocity=100 -> lower=-3.14 upper=3.14 effort=30 velocity=1000
- joint right_wheel_joint: limit lower=-3.14 upper=3.14 effort=100 velocity=100 -> effort=4.5 velocity=1000

Commit message: fix: align whole robot joint axes

File: resources/robots/wheel_legged_fyt_whole/urdf/wheel_legged_fyt_whole.urdf (robot description, URDF)
Before this commit: robot wheel_legged_fyt_whole, 7 links, 6 joints
Joints:
- joint left_leg_joint: axis 0 0 -1 -> 0 0 1
- joint right_leg_joint: axis 0 0 -1 -> 0 0 1

Commit message: chore: round whole robot inertial values

File: resources/robots/wheel_legged_fyt_whole/urdf/wheel_legged_fyt_whole.urdf (robot description, URDF)
Before this commit: robot wheel_legged_fyt_whole, 7 links, 6 joints
Links:
- link left_leg_link: mass 0.275645352077111 -> 0.3
